Commit message: fix for kuams

File: kuams_description/urdf/kuams.xacro (robot description, xacro)
@@ -196,5 +196,5 @@
     </link>
     <joint name="laser_joint" type="fixed">
-        <origin rpy="3.1415926535 0 0" xyz="0.5 0 0.4"/>
+        <origin rpy="3.1415926535 0 0" xyz="0.5 0 0.3"/>
         <parent link="base_link"/>
         <child link="laser"/>

Commit message: edit xacro file

File: kuams_description/urdf/kuams.xacro (robot description, xacro)
@@ -10,4 +10,5 @@
     <link name="base_floor">
         <visual>
+            <origin xyz="-0.08 0 0" rpy="0 0 0" />
             <geometry>
             	<mesh filename="file://$(find kuams_description)/meshes/KUAMS_ver.5.1.0.dae" />
@@ -19,4 +20,5 @@
         </visual>
         <collision>
+            <origin xyz="-0.08 0 0" rpy="0 0 0" />
             <geometry>
             	<mesh filename="file://$(find kuams_description)/meshes/KUAMS_ver.5.1.0.dae" />
@@ -47,6 +49,6 @@
                 <box size="0.250 0.260 0.050"/>
             </geometry>
-            <material name="grey">
-                <color rgba="0.5 0.5 0.5 1.0"/>
+            <material name="dark_grey">
+                <color rgba="0.1 0.1 0.1 1.0"/>
             </material>
         </visual>
@@ -70,6 +72,6 @@
             </geometry>
             <origin xyz="0 0 0" rpy="0 0 0" />
-            <material name="black">
-                <color rgba="0 0 0 1.0"/>
+            <material name="dark_grey">
+                <color rgba="0.1 0.1 0.1 1.0"/>
             </material>
         </visual>
@@ -103,6 +105,6 @@
                 <cylinder length="0.05" radius="0.1325"/>
             </geometry>
-            <material name="black">
-                <color rgba="0 0 0 1.0"/>
+            <material name="dark_grey">
+                <color rgba="0.1 0.1 0.1 1.0"/>
             </material>
         </visual>
@@ -129,6 +131,6 @@
                 <cylinder length="0.05" radius="0.1325"/>
             </geometry>
-            <material name="black">
-                <color rgba="0 0 0 1.0"/>
+            <material name="dark_grey">
+                <color rgba="0.1 0.1 0.1 1.0"/>
             </material>
         </visual>
@@ -157,6 +159,6 @@
                 <cylinder length="0.05" radius="0.1325"/>
             </geometry>
-            <material name="black">
-                <color rgba="0 0 0 1.0"/>
+            <material name="dark_grey">
+                <color rgba="0.1 0.1 0.1 1.0"/>
             </material>
         </visual>

Commit message: edit kuams xacro file

File: kuams_description/urdf/kuams.xacro (robot description, xacro)
@@ -10,8 +10,6 @@
     <link name="base_floor">
         <visual>
-            <origin xyz="-0.08 0 0" rpy="0 0 0" />
             <geometry>
             	<mesh filename="file://$(find kuams_description)/meshes/KUAMS_ver.5.1.0.dae" />
-                <!--<box size="0.600 0.400 0.050"/>-->
             </geometry>
             <material name="grey">
@@ -20,8 +18,6 @@
         </visual>
         <collision>
-            <origin xyz="-0.08 0 0" rpy="0 0 0" />
             <geometry>
             	<mesh filename="file://$(find kuams_description)/meshes/KUAMS_ver.5.1.0.dae" />
-                <!--<box size="0.600 0.400 0.050"/>-->
             </geometry>
         </collision>
@@ -40,24 +36,4 @@
     </joint>
     <link name="footrest_link">
-        <collision>
-            <geometry>
-                <box size="0.250 0.260 0.050"/>
-            </geometry>
-        </collision>
-        <visual>
-            <geometry>
-                <box size="0.250 0.260 0.050"/>
-            </geometry>
-            <material name="dark_grey">
-                <color rgba="0.1 0.1 0.1 1.0"/>
-            </material>
-        </visual>
-        <inertial>
-            <origin xyz="0 0 0" rpy="0 0 0" />
-            <mass value="1" />
-            <inertia ixx="1.0"  ixy="0.0"   ixz="0.0"
-                                iyy="1.0"   iyz="0.0"
-                                            izz="1.0" />
-        </inertial>
     </link>
     <joint name="footrest_joint" type="fixed">
@@ -190,5 +166,5 @@
     </link>
     <joint name="velodyne" type="fixed">
-        <origin rpy="0 0 0" xyz="0.1 0 0.8"/>
+        <origin rpy="0 0 0" xyz="0.2 0 0.8"/>
         <parent link="base_link"/>
         <child link="velodyne"/>
@@ -198,5 +174,5 @@
     </link>
     <joint name="laser_joint" type="fixed">
-        <origin rpy="3.1415926535 0 0" xyz="0.5 0 0.3"/>
+        <origin rpy="3.1415926535 0 0" xyz="0.6 0 0.3"/>
         <parent link="base_link"/>
         <child link="laser"/>
@@ -206,5 +182,5 @@
     </link>
     <joint name="gx5_25" type="fixed">
-        <origin rpy="0 0 0" xyz="0.1 0 0.75"/>
+        <origin rpy="0 0 0" xyz="0.2 0 0.75"/>
         <parent link="base_link"/>
         <child link="gx5_25"/>

Commit message: edit laser frame name

File: kuams_description/urdf/kuams.xacro (robot description, xacro)
@@ -171,10 +171,10 @@
     </joint>
     <!-- laser -->
-    <link name="laser">
+    <link name="livox_frame">
     </link>
     <joint name="laser_joint" type="fixed">
         <origin rpy="3.1415926535 0 0" xyz="0.6 0 0.3"/>
         <parent link="base_link"/>
-        <child link="laser"/>
+        <child link="livox_frame"/>
     </joint>
     <!-- gx5 -->

Commit message: add new sensor link

File: kuams_description/urdf/kuams.xacro (robot description, xacro)
@@ -170,10 +170,17 @@
         <child link="velodyne"/>
     </joint>
+    <link name="front_sensor_link">
+    </link>
+    <joint name="livox_front_sensor_joint" type="fixed">
+        <origin rpy="0 0 0" xyz="0.6 0 0.3"/>
+        <parent link="base_link"/>
+        <child link="front_sensor_link"/>
+    </joint>
     <!-- laser -->
     <link name="livox_frame">
     </link>
     <joint name="laser_joint" type="fixed">
-        <origin rpy="3.1415926535 0 0" xyz="0.6 0 0.3"/>
-        <parent link="base_link"/>
+        <origin rpy="3.1415926535 -0.34906585039886 0" xyz="0 0 0"/>
+        <parent link="front_sensor_link"/>
         <child link="livox_frame"/>
     </joint>

Commit message: update kuams.xacro

File: kuams_description/urdf/kuams.xacro (robot description, xacro)
@@ -1,52 +1,48 @@
 <?xml version="1.0"?>
 <robot xmlns:xacro="http://www.ros.org/wiki/xacro" name="kuams" >
-    <link name="base_link" />
-    <!-- <link name="base_footprint" />
-    <joint name="base_joint" type="fixed">
-        <parent link="base_footprint" />
-        <child link="base_link" />
-        <origin xyz="0 0 0.06625" rpy="0 0 0"/>
-    </joint> -->
+    <link name="base_link">
+        <visual>
+            <geometry>
+                <cylinder length="0.2" radius="0.01"/>
+            </geometry>
+            <material name="blue">
+                <color rgba="0.0 0.0 1.0 1.0"/>
+            </material>
+        </visual>
+    </link>
     <link name="base_floor">
         <visual>
             <geometry>
-            	<mesh filename="file://$(find kuams_description)/meshes/KUAMS_ver.5.1.0.dae" />
-            </geometry>
-            <material name="grey">
-                <color rgba="0.5 0.5 0.5 1.0"/>
-            </material>
-        </visual>
-        <collision>
-            <geometry>
-            	<mesh filename="file://$(find kuams_description)/meshes/KUAMS_ver.5.1.0.dae" />
-            </geometry>
-        </collision>
-        <inertial>
-            <origin xyz="0 0 0" rpy="0 0 0" />
-            <mass value="40" />
-            <inertia ixx="1.0"  ixy="0.0"   ixz="0.0"
-                                iyy="1.0"   iyz="0.0"
-                                            izz="1.0" />
-        </inertial>
-    </link>
-    <joint name="base_body_joint" type="fixed">
+                <box size="0.985 0.37 0.03"/>
+            </geometry>
+            <material name="grey">
+                <color rgba="0.5 0.5 0.5 1.0"/>
+            </material>
+        </visual>
+        <collision>
+            <geometry>
+                <box size="0.985 0.37 0.03"/>
+            </geometry>
+        </collision>
+        <inertial>
+            <origin xyz="0 0 0" rpy="0 0 0" />
+            <mass value="30" />
+            <inertia ixx="1.0"  ixy="0.0"   ixz="0.0"
+                                iyy="1.0"   iyz="0.0"
+                                            izz="1.0" />
+        </inertial>
+    </link>
+    <joint name="base_floor_joint" type="fixed">
         <parent link="base_link" />
         <child link="base_floor" />
-        <origin xyz="0.3 0 0.0" rpy="0 0 0"/>
-    </joint>
-    <link name="footrest_link">
-    </link>
-    <joint name="footrest_joint" type="fixed">
-        <parent link="base_floor" />
-        <child link="footrest_link" />
-        <origin xyz="0.320 0 0" rpy="0 0 0"/>
-    </joint>
-    <link name="left_wheel_link">
-        <visual>
-            <geometry>
-                <cylinder length="0.05" radius="0.1325"/>
-            </geometry>
-            <origin xyz="0 0 0" rpy="0 0 0" />
-            <material name="dark_grey">
+        <origin xyz="0.3 0 0" rpy="0 0 0"/>
+    </joint>
+    <link name="left_wheel">
+        <visual>
+            <geometry>
+                <cylinder length="0.05" radius="0.1325"/>
+            </geometry>
+            <origin xyz="0 0 0" rpy="0 0 0" />
+            <material name="black">
                 <color rgba="0.1 0.1 0.1 1.0"/>
             </material>
@@ -63,23 +59,23 @@
         </inertial>
     </link>
-    <joint name="leftWheel" type="continuous">
-        <parent link="base_floor" />
-        <child link="left_wheel_link" />
-        <origin xyz="-0.3 0.245 0" rpy="-1.57 0 0" />
+    <joint name="left_wheel_joint" type="continuous">
+        <parent link="base_floor" />
+        <child link="left_wheel" />
+        <origin xyz="-0.3 0.260 0.015" rpy="1.571 0 0" />
         <axis xyz="0 0 1" />
     </joint>
-    <link name="right_wheel_link">
-        <collision>
-            <origin xyz="0 0 0" rpy="0 0 0" />
-            <geometry>
-                <cylinder length="0.05" radius="0.1325"/>
-            </geometry>
-        </collision>
-        <visual>
-            <origin xyz="0 0 0" rpy="0 0 0" />
-            <geometry>
-                <cylinder length="0.05" radius="0.1325"/>
-            </geometry>
-            <material name="dark_grey">
+    <link name="right_wheel">
+        <collision>
+            <origin xyz="0 0 0" rpy="0 0 0" />
+            <geometry>
+                <cylinder length="0.05" radius="0.1325"/>
+            </geometry>
+        </collision>
+        <visual>
+            <origin xyz="0 0 0" rpy="0 0 0" />
+            <geometry>
+                <cylinder length="0.05" radius="0.1325"/>
+            </geometry>
+            <material name="black">
                 <color rgba="0.1 0.1 0.1 1.0"/>
             </material>
@@ -91,65 +87,199 @@
         </inertial>
     </link>
-    <joint name="rightWheel" type="continuous">
-        <parent link="base_floor" />
-        <child link="right_wheel_link" />
-        <origin xyz="-0.3 -0.245 0" rpy="1.57 0 0" />
+    <joint name="right_wheel_joint" type="continuous">
+        <parent link="base_floor" />
+        <child link="right_wheel" />
+        <origin xyz="-0.3 -0.260 0.015" rpy="-1.571 0 0" />
+        <axis xyz="0 0 -1" />
+    </joint>
+    <link name="left_front_wheel">
+        <collision>
+            <geometry>
+                <cylinder length="0.05" radius="0.1325"/>
+            </geometry>
+        </collision>
+        <visual>
+            <geometry>
+                <cylinder length="0.05" radius="0.1325"/>
+            </geometry>
+            <material name="black">
+                <color rgba="0.1 0.1 0.1 1.0"/>
+            </material>
+        </visual>
+        <inertial>
+            <origin xyz="0 0 0" rpy="0 0 0" />
+            <mass value="1.0" />
+            <inertia ixx="1.0"  ixy="0.0"   ixz="0.0"
+                                iyy="1.0"   iyz="0.0"
+                                            izz="1.0" />
+        </inertial>
+    </link>
+    <joint name="left_front_wheel_joint" type="fixed">
+        <parent link="base_floor" />
+        <child link="left_front_wheel" />
+        <origin xyz="0.330 -0.235 0" rpy="-1.571 0 0" />
+        <axis xyz="0 0 -1" />
+    </joint>
+    <link name="right_front_wheel">
+        <collision>
+            <geometry>
+                <cylinder length="0.05" radius="0.1325"/>
+            </geometry>
+        </collision>
+        <visual>
+            <geometry>
+                <cylinder length="0.05" radius="0.1325"/>
+            </geometry>
+            <material name="black">
+                <color rgba="0.1 0.1 0.1 1.0"/>
+            </material>
+        </visual>
+        <inertial>
+            <origin xyz="0 0 0" rpy="0 0 0" />
+            <mass value="1.0" />
+            <inertia ixx="1.0"  ixy="0.0"   ixz="0.0"
+                                iyy="1.0"   iyz="0.0"
+                                            izz="1.0" />
+        </inertial>
+    </link>
+    <joint name="right_front_wheel_joint" type="fixed">
+        <parent link="base_floor" />
+        <child link="right_front_wheel"/>
+        <origin xyz="0.330 0.235 0" rpy="1.571 0 0" />
         <axis xyz="0 0 1" />
     </joint>
-    <link name="frontwheel_left">
-        <collision>
-            <geometry>
-                <cylinder length="0.05" radius="0.1325"/>
-            </geometry>
-        </collision>
-        <visual>
-            <geometry>
-                <cylinder length="0.05" radius="0.1325"/>
-            </geometry>
-            <material name="dark_grey">
-                <color rgba="0.1 0.1 0.1 1.0"/>
-            </material>
-        </visual>
-        <inertial>
-            <origin xyz="0 0 0" rpy="0 0 0" />
-            <mass value="1.0" />
-            <inertia ixx="1.0"  ixy="0.0"   ixz="0.0"
-                                iyy="1.0"   iyz="0.0"
-                                            izz="1.0" />
-        </inertial>
-    </link>
-    <joint name="frontwheel_left_joint" type="fixed">
-        <parent link="base_floor" />
-        <child link="frontwheel_left" />
-        <origin xyz="0.3 -0.245 0" rpy="1.57 0 0" />
-        <axis xyz="0 0 1" />
-    </joint>
-    <link name="frontwheel_right">
-        <collision>
-            <geometry>
-                <cylinder length="0.05" radius="0.1325"/>
-            </geometry>
-        </collision>
-        <visual>
-            <geometry>
-                <cylinder length="0.05" radius="0.1325"/>
-            </geometry>
-            <material name="dark_grey">
-                <color rgba="0.1 0.1 0.1 1.0"/>
-            </material>
-        </visual>
-        <inertial>
-            <origin xyz="0 0 0" rpy="0 0 0" />
-            <mass value="1.0" />
-            <inertia ixx="1.0"  ixy="0.0"   ixz="0.0"
-                                iyy="1.0"   iyz="0.0"
-                                            izz="1.0" />
-        </inertial>
-    </link>
-    <joint name="frontwheel_right_joint" type="fixed">
-        <parent link="base_floor" />
-        <child link="frontwheel_right"/>
-        <origin xyz="0.3 0.245 0" rpy="1.57 0 0" />
-        <axis xyz="0 0 -1" />
+    <link name="seat">
+        <visual>
+            <geometry>
+                <box size="0.42 0.42 0.40"/>
+            </geometry>
+            <material name="grey">
+                <color rgba="0.5 0.5 0.5 1.0"/>
+            </material>
+        </visual>
+        <collision>
+            <geometry>
+                <box size="0.42 0.42 0.40"/>
+            </geometry>
+        </collision>
+        <inertial>
+            <origin xyz="0 0 0" rpy="0 0 0" />
+            <mass value="12" />
+            <inertia ixx="1.0"  ixy="0.0"   ixz="0.0"
+                                iyy="1.0"   iyz="0.0"
+                                            izz="1.0" />
+        </inertial>
+    </link>
+    <joint name="seat_joint" type="fixed">
+        <parent link="base_floor" />
+        <child link="seat" />
+        <origin xyz="-0.10 0 0.215" rpy="0 0 0"/>
+    </joint>
+    <link name="left_sensor_arm">
+        <collision>
+            <geometry>
+                <cylinder length="0.11" radius="0.013"/>
+            </geometry>
+        </collision>
+        <visual>
+            <geometry>
+                <cylinder length="0.11" radius="0.013"/>
+            </geometry>
+            <material name="grey">
+                <color rgba="0.5 0.5 0.5 1.0"/>
+            </material>
+        </visual>
+    </link>
+    <joint name="left_sensor_arm_joint" type="fixed">
+        <parent link="seat"/>
+        <child link="left_sensor_arm"/>
+        <origin xyz="0.20 0.235 0.07" rpy="0 0 0"/>
+    </joint>
+    <link name="right_sensor_arm">
+        <collision>
+            <geometry>
+                <cylinder length="0.11" radius="0.013"/>
+            </geometry>
+        </collision>
+        <visual>
+            <geometry>
+                <cylinder length="0.11" radius="0.013"/>
+            </geometry>
+            <material name="grey">
+                <color rgba="0.5 0.5 0.5 1.0"/>
+            </material>
+        </visual>
+    </link>
+    <joint name="right_sensor_arm_joint" type="fixed">
+        <parent link="seat"/>
+        <child link="right_sensor_arm"/>
+        <origin xyz="0.20 -0.235 0.07" rpy="0 0 0"/>
+    </joint>
+    <link name="backrest">
+        <visual>
+            <geometry>
+                <box size="0.10 0.42 0.72"/>
+            </geometry>
+            <material name="grey">
+                <color rgba="0.5 0.5 0.5 1.0"/>
+            </material>
+        </visual>
+        <collision>
+            <geometry>
+                <box size="0.10 0.42 0.72"/>
+            </geometry>
+        </collision>
+        <inertial>
+            <origin xyz="0 0 0" rpy="0 0 0" />
+            <mass value="7" />
+            <inertia ixx="1.0"  ixy="0.0"   ixz="0.0"
+                                iyy="1.0"   iyz="0.0"
+                                            izz="1.0" />
+        </inertial>
+    </link>
+    <joint name="backrest_joint" type="fixed">
+        <parent link="base_floor" />
+        <child link="backrest" />
+        <origin xyz="-0.36 0 0.375" rpy="0 0 0"/>
+    </joint>
+    <link name="left_arm">
+        <visual>
+            <geometry>
+                <box size="0.09 0.07 0.535"/>
+            </geometry>
+            <material name="grey">
+                <color rgba="0.5 0.5 0.5 1.0"/>
+            </material>
+        </visual>
+        <collision>
+            <geometry>
+                <box size="0.09 0.07 0.535"/>
+            </geometry>
+        </collision>
+    </link>
+    <joint name="left_arm_joint" type="fixed">
+        <parent link="seat" />
+        <child link="left_arm" />
+        <origin xyz="0 0.245 0.30" rpy="0 1.0 0"/>
+    </joint>
+    <link name="right_arm">
+        <visual>
+            <geometry>
+                <box size="0.09 0.07 0.535"/>
+            </geometry>
+            <material name="grey">
+                <color rgba="0.5 0.5 0.5 1.0"/>
+            </material>
+        </visual>
+        <collision>
+            <geometry>
+                <box size="0.09 0.07 0.535"/>
+            </geometry>
+        </collision>
+    </link>
+    <joint name="right_arm_joint" type="fixed">
+        <parent link="seat" />
+        <child link="right_arm" />
+        <origin xyz="0 -0.245 0.30" rpy="0 1.0 0"/>
     </joint>
     <!-- IMU -->
