Commit message: adjusted for 2026-nakanoshima

File: kuams_description/urdf/kuams.xacro (robot description, xacro)
@@ -1,191 +1,189 @@
-<?xml version="1.0"?>
-<robot xmlns:xacro="http://www.ros.org/wiki/xacro" name="kuams" >
-    <link name="base_link">
-        <visual>
-            <geometry>
-                <cylinder length="0.2" radius="0.01"/>
-            </geometry>
-            <material name="blue">
-                <color rgba="0.0 0.0 1.0 1.0"/>
-            </material>
-        </visual>
+<?xml version="1.0" ?>
+<!-- =================================================================================== -->
+<!-- |    This document was autogenerated by xacro from /home/keisoku/kuams_dev_ws/install/kuams_description/share/kuams_description/urdf/kuams.xacro | -->
+<!-- |    EDITING THIS FILE BY HAND IS NOT RECOMMENDED                                 | -->
+<!-- =================================================================================== -->
+<robot name="kuams">
+  <link name="base_link">
+    <visual>
+      <geometry>
+        <cylinder length="0.2" radius="0.01"/>
+      </geometry>
+      <material name="blue">
+        <color rgba="0.0 0.0 1.0 1.0"/>
+      </material>
+    </visual>
+  </link>
+  <link name="base_floor">
+    <visual>
+      <geometry>
+        <mesh filename="file:///home/keisoku/kuams_dev_ws/install/kuams_description/share/kuams_description/meshes/KUAMS_ver.5.1.0.dae"/>
+      </geometry>
+      <material name="grey">
+        <color rgba="0.5 0.5 0.5 1.0"/>
+      </material>
+    </visual>
+    <collision>
+      <geometry>
+        <mesh filename="file:///home/keisoku/kuams_dev_ws/install/kuams_description/share/kuams_description/meshes/KUAMS_ver.5.1.0.dae"/>
+      </geometry>
+    </collision>
+    <inertial>
+      <origin rpy="0 0 0" xyz="0 0 0"/>
+      <mass value="30"/>
+      <inertia ixx="1.0" ixy="0.0" ixz="0.0" iyy="1.0" iyz="0.0" izz="1.0"/>
+    </inertial>
+  </link>
+  <joint name="base_floor_joint" type="fixed">
+    <parent link="base_link"/>
+    <child link="base_floor"/>
+    <origin rpy="0 0 0" xyz="0.3 0 0"/>
+  </joint>
+  <link name="left_wheel">
+    <visual>
+      <geometry>
+        <cylinder length="0.05" radius="0.1325"/>
+      </geometry>
+      <origin rpy="0 0 0" xyz="0 0 0"/>
+      <material name="black">
+        <color rgba="0.1 0.1 0.1 1.0"/>
+      </material>
+    </visual>
+    <collision>
+      <geometry>
+        <cylinder length="0.05" radius="0.1325"/>
+      </geometry>
+    </collision>
+    <inertial>
+      <origin xyz="0 0 0"/>
+      <mass value="0.500"/>
+      <inertia ixx="0.0013541667" ixy="0" ixz="0" iyy="0.0013541667" iyz="0" izz="0.0025"/>
+    </inertial>
+  </link>
+  <joint name="left_wheel_joint" type="continuous">
+    <parent link="base_floor"/>
+    <child link="left_wheel"/>
+    <origin rpy="1.571 0 0" xyz="-0.3 0.260 0.015"/>
+    <axis xyz="0 0 1"/>
+  </joint>
+  <link name="right_wheel">
+    <collision>
+      <origin rpy="0 0 0" xyz="0 0 0"/>
+      <geometry>
+        <cylinder length="0.05" radius="0.1325"/>
+      </geometry>
+    </collision>
+    <visual>
+      <origin rpy="0 0 0" xyz="0 0 0"/>
+      <geometry>
+        <cylinder length="0.05" radius="0.1325"/>
+      </geometry>
+      <material name="black">
+        <color rgba="0.1 0.1 0.1 1.0"/>
+      </material>
+    </visual>
+    <inertial>
+      <origin xyz="0 0 0"/>
+      <mass value="0.500"/>
+      <inertia ixx="0.0013541667" ixy="0" ixz="0" iyy="0.0013541667" iyz="0" izz="0.0025"/>
+    </inertial>
+  </link>
+  <joint name="right_wheel_joint" type="continuous">
+    <parent link="base_floor"/>
+    <child link="right_wheel"/>
+    <origin rpy="-1.571 0 0" xyz="-0.3 -0.260 0.015"/>
+    <axis xyz="0 0 -1"/>
+  </joint>
+  <link name="left_front_wheel">
+    <collision>
+      <geometry>
+        <cylinder length="0.05" radius="0.1325"/>
+      </geometry>
+    </collision>
+    <visual>
+      <geometry>
+        <cylinder length="0.05" radius="0.1325"/>
+      </geometry>
+      <material name="black">
+        <color rgba="0.1 0.1 0.1 1.0"/>
+      </material>
+    </visual>
+    <inertial>
+      <origin rpy="0 0 0" xyz="0 0 0"/>
+      <mass value="1.0"/>
+      <inertia ixx="1.0" ixy="0.0" ixz="0.0" iyy="1.0" iyz="0.0" izz="1.0"/>
+    </inertial>
+  </link>
+  <joint name="left_front_wheel_joint" type="fixed">
+    <parent link="base_floor"/>
+    <child link="left_front_wheel"/>
+    <origin rpy="-1.571 0 0" xyz="0.330 -0.235 0"/>
+    <axis xyz="0 0 -1"/>
+  </joint>
+  <link name="right_front_wheel">
+    <collision>
+      <geometry>
+        <cylinder length="0.05" radius="0.1325"/>
+      </geometry>
+    </collision>
+    <visual>
+      <geometry>
+        <cylinder length="0.05" radius="0.1325"/>
+      </geometry>
+      <material name="black">
+        <color rgba="0.1 0.1 0.1 1.0"/>
+      </material>
+    </visual>
+    <inertial>
+      <origin rpy="0 0 0" xyz="0 0 0"/>
+      <mass value="1.0"/>
+      <inertia ixx="1.0" ixy="0.0" ixz="0.0" iyy="1.0" iyz="0.0" izz="1.0"/>
+    </inertial>
+  </link>
+  <joint name="right_front_wheel_joint" type="fixed">
+    <parent link="base_floor"/>
+    <child link="right_front_wheel"/>
+    <origin rpy="1.571 0 0" xyz="0.330 0.235 0"/>
+    <axis xyz="0 0 1"/>
+  </joint>
+  <!-- IMU -->
+  <link name="imu">
     </link>
-    <link name="base_floor">
-        <visual>
-            <geometry>
-            	<mesh filename="file://$(find kuams_description)/meshes/KUAMS_ver.5.1.0.dae" />
-            </geometry>
-            <material name="grey">
-                <color rgba="0.5 0.5 0.5 1.0"/>
-            </material>
-        </visual>
-        <collision>
-            <geometry>
-            	<mesh filename="file://$(find kuams_description)/meshes/KUAMS_ver.5.1.0.dae" />
-            </geometry>
-        </collision>
-        <inertial>
-            <origin xyz="0 0 0" rpy="0 0 0" />
-            <mass value="30" />
-            <inertia ixx="1.0"  ixy="0.0"   ixz="0.0"
-                                iyy="1.0"   iyz="0.0"
-                                            izz="1.0" />
-        </inertial>
+  <joint name="imu_joint" type="fixed">
+    <axis xyz="0 1 0"/>
+    <origin rpy="0 0.85521133347 3.14159265359" xyz="0.02 0 0.05"/>
+    <parent link="base_link"/>
+    <child link="imu"/>
+  </joint>
+  <!-- Velodyne -->
+  <link name="velodyne">
     </link>
-    <joint name="base_floor_joint" type="fixed">
-        <parent link="base_link" />
-        <child link="base_floor" />
-        <origin xyz="0.3 0 0" rpy="0 0 0"/>
-    </joint>
-    <link name="left_wheel">
-        <visual>
-            <geometry>
-                <cylinder length="0.05" radius="0.1325"/>
-            </geometry>
-            <origin xyz="0 0 0" rpy="0 0 0" />
-            <material name="black">
-                <color rgba="0.1 0.1 0.1 1.0"/>
-            </material>
-        </visual>
-        <collision>
-            <geometry>
-                <cylinder length="0.05" radius="0.1325"/>
-            </geometry>
-        </collision>
-        <inertial>
-            <origin xyz="0 0 0"/>
-            <mass value="0.500"/>
-            <inertia ixx="0.0013541667" ixy="0" ixz="0" iyy="0.0013541667" iyz="0" izz="0.0025"/>
-        </inertial>
+  <joint name="velodyne" type="fixed">
+    <origin rpy="0 0 0" xyz="0.2 0 0.8"/>
+    <parent link="base_link"/>
+    <child link="velodyne"/>
+  </joint>
+  <link name="front_sensor_link">
     </link>
-    <joint name="left_wheel_joint" type="continuous">
-        <parent link="base_floor" />
-        <child link="left_wheel" />
-        <origin xyz="-0.3 0.260 0.015" rpy="1.571 0 0" />
-        <axis xyz="0 0 1" />
-    </joint>
-    <link name="right_wheel">
-        <collision>
-            <origin xyz="0 0 0" rpy="0 0 0" />
-            <geometry>
-                <cylinder length="0.05" radius="0.1325"/>
-            </geometry>
-        </collision>
-        <visual>
-            <origin xyz="0 0 0" rpy="0 0 0" />
-            <geometry>
-                <cylinder length="0.05" radius="0.1325"/>
-            </geometry>
-            <material name="black">
-                <color rgba="0.1 0.1 0.1 1.0"/>
-            </material>
-        </visual>
-        <inertial>
-            <origin xyz="0 0 0"/>
-            <mass value="0.500"/>
-            <inertia ixx="0.0013541667" ixy="0" ixz="0" iyy="0.0013541667" iyz="0" izz="0.0025"/>
-        </inertial>
+  <joint name="livox_front_sensor_joint" type="fixed">
+    <origin rpy="0 0 0" xyz="0.6 0 0.3"/>
+    <parent link="base_link"/>
+    <child link="front_sensor_link"/>
+  </joint>
+  <!-- laser -->
+  <link name="livox_frame">
     </link>
-    <joint name="right_wheel_joint" type="continuous">
-        <parent link="base_floor" />
-        <child link="right_wheel" />
-        <origin xyz="-0.3 -0.260 0.015" rpy="-1.571 0 0" />
-        <axis xyz="0 0 -1" />
-    </joint>
-    <link name="left_front_wheel">
-        <collision>
-            <geometry>
-                <cylinder length="0.05" radius="0.1325"/>
-            </geometry>
-        </collision>
-        <visual>
-            <geometry>
-                <cylinder length="0.05" radius="0.1325"/>
-            </geometry>
-            <material name="black">
-                <color rgba="0.1 0.1 0.1 1.0"/>
-            </material>
-        </visual>
-        <inertial>
-            <origin xyz="0 0 0" rpy="0 0 0" />
-            <mass value="1.0" />
-            <inertia ixx="1.0"  ixy="0.0"   ixz="0.0"
-                                iyy="1.0"   iyz="0.0"
-                                            izz="1.0" />
-        </inertial>
+  <joint name="laser_joint" type="fixed">
+    <origin rpy="3.1415926535 -0.34906585039886 0" xyz="0 0 0"/>
+    <parent link="front_sensor_link"/>
+    <child link="livox_frame"/>
+  </joint>
+  <!-- gx5 -->
+  <link name="gx5_25">
     </link>
-    <joint name="left_front_wheel_joint" type="fixed">
-        <parent link="base_floor" />
-        <child link="left_front_wheel" />
-        <origin xyz="0.330 -0.235 0" rpy="-1.571 0 0" />
-        <axis xyz="0 0 -1" />
-    </joint>
-    <link name="right_front_wheel">
-        <collision>
-            <geometry>
-                <cylinder length="0.05" radius="0.1325"/>
-            </geometry>
-        </collision>
-        <visual>
-            <geometry>
-                <cylinder length="0.05" radius="0.1325"/>
-            </geometry>
-            <material name="black">
-                <color rgba="0.1 0.1 0.1 1.0"/>
-            </material>
-        </visual>
-        <inertial>
-            <origin xyz="0 0 0" rpy="0 0 0" />
-            <mass value="1.0" />
-            <inertia ixx="1.0"  ixy="0.0"   ixz="0.0"
-                                iyy="1.0"   iyz="0.0"
-                                            izz="1.0" />
-        </inertial>
-    </link>
-    <joint name="right_front_wheel_joint" type="fixed">
-        <parent link="base_floor" />
-        <child link="right_front_wheel"/>
-        <origin xyz="0.330 0.235 0" rpy="1.571 0 0" />
-        <axis xyz="0 0 1" />
-    </joint>
-    <!-- IMU -->
-    <link name="imu">
-    </link>
-    <joint name="imu_joint" type="fixed">
-        <axis xyz="0 1 0" />
-        <origin xyz="0.02 0 0.05" rpy="0 0.85521133347 3.14159265359"/>
-        <parent link="base_link"/>
-        <child link="imu"/>
-    </joint>
-    <!-- Velodyne -->
-    <link name="velodyne">
-    </link>
-    <joint name="velodyne" type="fixed">
-        <origin rpy="0 0 0" xyz="0.2 0 0.8"/>
-        <parent link="base_link"/>
-        <child link="velodyne"/>
-    </joint>
-    <link name="front_sensor_link">
-    </link>
-    <joint name="livox_front_sensor_joint" type="fixed">
-        <origin rpy="0 0 0" xyz="0.6 0 0.3"/>
-        <parent link="base_link"/>
-        <child link="front_sensor_link"/>
-    </joint>
-    <!-- laser -->
-    <link name="livox_frame">
-    </link>
-    <joint name="laser_joint" type="fixed">
-        <origin rpy="3.1415926535 -0.34906585039886 0" xyz="0 0 0"/>
-        <parent link="front_sensor_link"/>
-        <child link="livox_frame"/>
-    </joint>
-    <!-- gx5 -->
-    <link name="gx5_25">
-    </link>
-    <joint name="gx5_25" type="fixed">
-        <origin rpy="0 0 0" xyz="0.2 0 0.75"/>
-        <parent link="base_link"/>
-        <child link="gx5_25"/>
-    </joint>
+  <joint name="gx5_25" type="fixed">
+    <origin rpy="0 0 0" xyz="0.2 0 0.75"/>
+    <parent link="base_link"/>
+    <child link="gx5_25"/>
+  </joint>
 </robot>
